File: Voltlog TagConnect Adapter.kicad_pcb (KiCad board)
At the start: 2 copper layers, 50 x 62 mm, 23 parts, among them J1 VoltLink_target, J2 JTAG 10pin P1.27mm, J3 TC2030-IDC 6-Pin, J4 TC2050-IDC 10-Pin, J5 Conn_ARM_JTAG_SWD_20

Commit message: Update
Sample PCB
Parts:
- removed REF**: Fiducial_0.5mm_Mask1mm, Fiducial:Fiducial_0.5mm_Mask1mm
- J5: footprint Connector_IDC:IDC-Header_2x20_P2.54mm_Vertical_SMD -> Connector_IDC:IDC-Header_2x10_P2.54mm_Vertical_SMD
- moved J5 12.6 mm to (148.7, 81.9)
- moved kibuzzard-64FC2395 9.50 mm to (149.0, 101.0), turned to 0 degrees
- moved V1 0.50 mm to (121.5, 94.5)
Other:
- board text added: "J-Link"
- board text added: "ST-LINK Black Magic Cortex"
- board text added: "TC2030 6-Pin"
- board text added: "TC2050 10-Pin"
- board text added: "Updated Version"
- board text removed: "FIRST EDITION"
- board text removed: "JLCJLCJLCJLC"
