File: Voltlog TagConnect Adapter.kicad_sch (KiCad schematic)
At the start: 10 parts, among them J1 JTAG 10pin P1.27mm, J1 TC2050-IDC 10-Pin, J3 TC2030-IDC 6-Pin, J3 VoltLink_target, J5 Conn_ARM_JTAG_SWD_20

Commit message: Update
Sample PCB
Parts:
- J5: footprint Connector_IDC:IDC-Header_2x20_P2.54mm_Vertical_SMD -> Connector_IDC:IDC-Header_2x10_P2.54mm_Vertical_SMD
